File: 3_21_22/OPLL01/OPLL01.kicad_pcb (KiCad board)
At the start: 2 copper layers, 101.6 x 53.3 mm, 13 parts, among them P1 Digital, P10 CONN_01X01, P11 CONN_01X01, P12 CONN_01X01, P13 CONN_01X01, P2 Power, P3 Analog, P4 Analog, P5 PWM, P6 PWM, P7 Communication, P8 CONN_01X01, P9 CONN_01X01

Commit message: Update OPLL
Parts:
- added C1: 10uF, Capacitor_SMD:C_0805_2012Metric, F.Cu at (155.3, 94.6)
- added C2: 15nF, Capacitor_SMD:C_0805_2012Metric, F.Cu at (144.3, 101.8)
- added C3: 10uF, Capacitor_SMD:C_0805_2012Metric, F.Cu at (160.0, 87.7)
- added C4: 15pF, Capacitor_SMD:C_0805_2012Metric, F.Cu at (155.3, 91.6)
- added C5: 15pF, Capacitor_SMD:C_0805_2012Metric, F.Cu at (144.3, 104.8)
- added C6: 1000uF, Capacitor_SMD:CP_Elec_10x10, F.Cu at (130.4, 106.5)
- added C7: 100nF, Capacitor_SMD:C_0805_2012Metric, F.Cu at (148.7, 101.8)
- added J1: AudioJack3, 3K:PJ-320B, F.Cu at (103.6, 109.0)
- added L1: 1mH, Inductor_SMD:L_0805_2012Metric, F.Cu at (160.0, 84.8)
- added R1: 2k2, Resistor_SMD:R_0805_2012Metric, F.Cu at (159.9, 90.6)
- added R2: 4k7, Resistor_SMD:R_0805_2012Metric, F.Cu at (144.2, 107.8)
- added R3: 2k2, Resistor_SMD:R_0805_2012Metric, F.Cu at (148.7, 104.8)
- added R4: 10K, Resistor_SMD:R_0805_2012Metric, F.Cu at (155.2, 97.5)
- added R5: 4k7, Resistor_SMD:R_0805_2012Metric, F.Cu at (153.2, 101.7)
- added U1: LMC660AIM, Package_SO:SOIC-14_3.9x8.7mm_P1.27mm, F.Cu at (148.8, 95.2)
- added U2: YM2413, Package_DIP:DIP-18_W7.62mm, F.Cu at (120.8, 86.7)
- added Y1: 3.57MHz, Crystal:Crystal_HC49-4H_Vertical, F.Cu at (148.7, 86.7)
Connections:
- P1 pad 10: /47 -> (no net)
- P1 pad 11: /44 -> (no net)
- P1 pad 12: /45 -> (no net)
- P1 pad 13: /42 -> (no net)
- P1 pad 14: /43 -> (no net)
- P1 pad 15: /40 -> (no net)
- P1 pad 16: /41 -> (no net)
- P1 pad 17: /38 -> (no net)
- P1 pad 18: /39 -> (no net)
- P1 pad 19: /36 -> (no net)
- P1 pad 20: /37 -> (no net)
- P1 pad 21: /34 -> (no net)
- P1 pad 22: /35 -> (no net)
- P1 pad 23: /32 -> (no net)
- P1 pad 24: /33 -> (no net)
- P1 pad 25: /30 -> (no net)
- P1 pad 26: /31 -> (no net)
- P1 pad 27: /28 -> (no net)
- P1 pad 28: /29 -> (no net)
- P1 pad 29: /26 -> (no net)
- P1 pad 3: /52(SCK) -> (no net)
- P1 pad 30: /27 -> (no net)
- P1 pad 31: /24 -> (no net)
- P1 pad 32: /25 -> (no net)
- P1 pad 33: /22 -> (no net)
- P1 pad 34: /23 -> (no net)
- P1 pad 4: /53(SS) -> (no net)
- P1 pad 5: /50(MISO) -> (no net)
- P1 pad 6: /51(MOSI) -> (no net)
- P1 pad 7: /48 -> (no net)
- P1 pad 8: /49 -> (no net)
- P1 pad 9: /46 -> (no net)
- P10 pad 1: Net-(P10-Pad1) -> (no net)
- P11 pad 1: Net-(P11-Pad1) -> (no net)
- P12 pad 1: Net-(P12-Pad1) -> (no net)
- P13 pad 1: Net-(P13-Pad1) -> (no net)
- P2 pad 1: Net-(P2-Pad1) -> (no net)
- P2 pad 2: /IOREF -> (no net)
- P2 pad 3: /Reset -> (no net)
- P2 pad 4: +3V3 -> (no net)
- P2 pad 8: /Vin -> (no net)
- P3 pad 2: /A1 -> /~CS
- P3 pad 3: /A2 -> /~IC
- P3 pad 4: /A3 -> /~WE
- P3 pad 5: /A4 -> (no net)
- P3 pad 6: /A5 -> (no net)
- P3 pad 7: /A6 -> (no net)
- P3 pad 8: /A7 -> (no net)
- P4 pad 1: /A8 -> /D0
- P4 pad 2: /A9 -> /D1
- P4 pad 3: /A10 -> /D2
- P4 pad 4: /A11 -> /D3
- P4 pad 5: /A12 -> /D4
- P4 pad 6: /A13 -> /D5
- P4 pad 7: /A14 -> /D6
- P4 pad 8: /A15 -> /D7
- P5 pad 1: /SCL -> (no net)
- P5 pad 10: /8(**) -> (no net)
- P5 pad 2: /SDA -> (no net)
- P5 pad 3: /AREF -> (no net)
- P5 pad 5: /13(**) -> (no net)
- P5 pad 6: /12(**) -> (no net)
- P5 pad 7: /11(**) -> (no net)
- P5 pad 8: /10(**) -> (no net)
- P5 pad 9: /9(**) -> (no net)
- P6 pad 1: /7(**) -> (no net)
- P6 pad 2: /6(**) -> (no net)
- P6 pad 3: /5(**) -> (no net)
- P6 pad 4: /4(**) -> (no net)
- P6 pad 5: /3(**) -> (no net)
- P6 pad 6: /2(**) -> (no net)
- P6 pad 7: /1(Tx0) -> (no net)
- P6 pad 8: /0(Rx0) -> (no net)
- P7 pad 1: /14(Tx3) -> (no net)
- P7 pad 2: /15(Rx3) -> (no net)
- P7 pad 3: /16(Tx2) -> (no net)
- P7 pad 4: /17(Rx2) -> (no net)
- P7 pad 5: /18(Tx1) -> (no net)
- P7 pad 6: /19(Rx1) -> (no net)
- P7 pad 7: /20(SDA) -> (no net)
- P7 pad 8: /21(SCL) -> (no net)
- P8 pad 1: Net-(P8-Pad1) -> (no net)
- P9 pad 1: Net-(P9-Pad1) -> (no net)
