File: 3_21_22/OPLL01/OPLL01.kicad_pcb (KiCad board)
At the start: 2 copper layers, 101.6 x 53.3 mm, 30 parts, among them J1 AudioJack3, P1 Digital, P10 CONN_01X01, P11 CONN_01X01, P12 CONN_01X01, P13 CONN_01X01, P2 Power, P3 Analog, P4 Analog, P5 PWM, P6 PWM, P7 Communication, P8 CONN_01X01, P9 CONN_01X01, U1 LMC660AIM, U2 YM2413, Y1 3.57MHz

Commit message: End of OPLL Project
finished routing
Parts:
- moved C6 62.7 mm to (189.3, 85.2)
- moved C3 45.9 mm to (117.6, 105.2)
- moved U2 43.8 mm to (157.8, 110.2), turned to 180 degrees
- moved C1 41.8 mm to (117.6, 112.6)
- moved L1 27.6 mm to (186.5, 77.2), turned to 180 degrees
- moved C5 27.2 mm to (165.8, 88.1), turned to 270 degrees
- moved R4 26.8 mm to (179.0, 85.3)
- moved R5 26.0 mm to (166.0, 79.2), turned to 270 degrees
- moved R1 17.4 mm to (147.3, 102.6)
- moved Y1 15.1 mm to (161.9, 94.1), turned to 90 degrees
- moved R2 13.9 mm to (133.6, 98.7), turned to 270 degrees
- moved C2 12.7 mm to (133.5, 95.1), turned to 90 degrees
- moved C4 11.0 mm to (165.7, 95.0), turned to 90 degrees
- moved U1 9.95 mm to (139.1, 97.3)
- moved R3 4.75 mm to (147.3, 100.2)
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Connections:
- net Net-(C6-Pad1) renamed /VC
Routing:
- net +5V: track 0.00 -> 122.8 mm, vias 0 -> 4
- net VREF: track 0.00 -> 49.2 mm
- net /D7: track 0.00 -> 47.9 mm
- net /D6: track 0.00 -> 43.4 mm
- net /D5: track 0.00 -> 39.9 mm
- net /D4: track 0.00 -> 36.3 mm
- net /D0: track 0.00 -> 35.1 mm
- net Net-(C1-Pad2): track 0.00 -> 34.2 mm
- net /D1: track 0.00 -> 33.1 mm
- net /D3: track 0.00 -> 32.7 mm
- net /A0: track 0.00 -> 32.6 mm
- net /~WE: track 0.00 -> 31.5 mm
- net /D2: track 0.00 -> 29.1 mm
- net /~CS: track 0.00 -> 27.9 mm
- net Net-(C3-Pad2): track 0.00 -> 26.1 mm, vias 0 -> 2
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- added copper zone on B.Cu, net GND
- added copper zone on F.Cu, net GND
Other:
- net class Default: trace_width 0.25 -> 0.4; via_drill 0.4 -> 0.3
- net class PWR added: clearance 0.2, trace_width 0.6, via_dia 0.6, via_drill 0.3
