File: 3_21_22/OPLL01/OPLL01.sch (KiCad schematic (older format))
At the start: 30 parts, among them J1 AudioJack3, P1 Digital, P10 CONN_01X01, P11 CONN_01X01, P12 CONN_01X01, P13 CONN_01X01, P2 Power, P3 Analog, P4 Analog, P5 PWM, P6 PWM, P7 Communication, P8 CONN_01X01, P9 CONN_01X01, U1 LMC660AIM, U2 YM2413, Y1 3.57MHz

Commit message: Update OPLL
Parts:
- C1, C2, C3, C4, C5, C7: footprint (none) -> Capacitor_SMD:C_0805_2012Metric
- C6: footprint (none) -> Capacitor_SMD:CP_Elec_10x10
- J1: footprint (none) -> 3K:PJ-320B
- L1: footprint (none) -> Inductor_SMD:L_0805_2012Metric
- R1, R2, R3, R4, R5: footprint (none) -> Resistor_SMD:R_0805_2012Metric
- U1: footprint (none) -> Package_SO:SOIC-14_3.9x8.7mm_P1.27mm
- Y1: footprint (none) -> Crystal:Crystal_HC49-4H_Vertical
Connections:
- net labels added: CTRL_BUS, D0, D1, D2, D3, D4, D5, D6, D7, DATA_BUS, ~CS, ~IC, ~WE
- net labels removed: A1, A10, A11, A12, A13, A14, A15, A2, A3, A8, A9
- wire segments 151 -> 175
