File: 3_21_22/OPLL01/OPLL01.sch (KiCad schematic (older format))
At the start: 30 parts, among them J1 AudioJack3, P1 Digital, P10 CONN_01X01, P11 CONN_01X01, P12 CONN_01X01, P13 CONN_01X01, P2 Power, P3 Analog, P4 Analog, P5 PWM, P6 PWM, P7 Communication, P8 CONN_01X01, P9 CONN_01X01, U1 LMC660AIM, U2 YM2413, Y1 3.57MHz

Commit message: End of OPLL Project
finished routing
Connections:
- net labels added: VC
Changed lines of the file:
@@
 Wire Bus Line
 	1250 2100 1250 3150
+Text Label 4900 5200 0    50   ~ 0
+VC
 $EndSCHEMATC
