File: 3_21_22/Protoino01/Protoino01.kicad_pcb (KiCad board)
At the start: 2 copper layers, 0 parts

Commit message: Protoino - 14.10.2021
Parts:
- added C1: 100nF, Capacitor_SMD:C_0603_1608Metric, F.Cu at (313.8, 98.5)
- added C10: 100nF, Capacitor_SMD:C_0603_1608Metric, F.Cu at (313.8, 100.2)
- added C11: 100nF, Capacitor_SMD:C_0603_1608Metric, F.Cu at (299.9, 97.7)
- added C2: 100nF, Capacitor_SMD:C_0603_1608Metric, F.Cu at (207.6, 104.8)
- added C3: 10uF, Capacitor_SMD:C_0805_2012Metric, F.Cu at (209.6, 104.9)
- added C4: 100nF, Capacitor_SMD:C_0603_1608Metric, F.Cu at (246.6, 102.3)
- added C5: 15pF, Capacitor_SMD:C_0603_1608Metric, F.Cu at (297.0, 102.8)
- added C6: 15pF, Capacitor_SMD:C_0603_1608Metric, F.Cu at (299.6, 106.0)
- added C7: 100nF, Capacitor_SMD:C_0603_1608Metric, F.Cu at (299.9, 99.6)
- added C8: 10uF, Capacitor_SMD:C_0805_2012Metric, F.Cu at (298.4, 95.9)
- added C9: 100nF, Capacitor_SMD:C_0603_1608Metric, F.Cu at (253.6, 96.9)
- added D1: PWR_Blue, LED_SMD:LED_0603_1608Metric, F.Cu at (204.7, 102.2)
- added F1: 700mA, Fuse:Fuse_0603_1608Metric, F.Cu at (204.7, 105.9)
- added FB1: Ferrite_Bead_Small, Inductor_SMD:L_0805_2012Metric, F.Cu at (205.0, 104.1)
- added H1: MountingHole_Pad, MountingHole:MountingHole_3mm_Pad, F.Cu at (199.9, 153.5)
- added H2: MountingHole_Pad, MountingHole:MountingHole_3mm_Pad, F.Cu at (332.9, 38.8)
- added H3: MountingHole_Pad, MountingHole:MountingHole_3mm_Pad, F.Cu at (332.9, 153.5)
- added H4: MountingHole_Pad, MountingHole:MountingHole_3mm_Pad, F.Cu at (199.9, 38.8)
- added J1: USB_C_Receptacle_USB2.0, Connector_USB:USB_C_Receptacle_HRO_TYPE-C-31-M-12, F.Cu at (201.1, 113.2)
- added J2: ICSP, Connector_PinHeader_2.54mm:PinHeader_2x03_P2.54mm_Vertical, F.Cu at (316.4, 110.0)
- added OLED1: I2C_OLED_128x64, IU10b:OLED_I2C_128x64, F.Cu at (306.5, 48.4)
- added R1: 4.7K, Resistor_SMD:R_0603_1608Metric, F.Cu at (311.5, 41.3)
- added R2: 4.7K, Resistor_SMD:R_0603_1608Metric, F.Cu at (307.1, 41.0)
- added R3: 5.1K, Resistor_SMD:R_0603_1608Metric, F.Cu at (209.5, 112.0)
- added R4: 5.1K, Resistor_SMD:R_0603_1608Metric, F.Cu at (209.5, 115.0)
- added R5: 2.2K, Resistor_SMD:R_0603_1608Metric, F.Cu at (207.9, 102.1)
- added U1: ATmega328P-AU, Package_QFP:TQFP-32_7x7mm_P0.8mm, F.Cu at (306.8, 98.5)
- added U2: CH340C, Package_SO:SOIC-16_3.9x9.9mm_P1.27mm, F.Cu at (251.9, 103.0)
- added Y1: 16MHz, Crystal:Crystal_SMD_3225-4Pin_3.2x2.5mm, F.Cu at (299.6, 103.1)

Commit message: protoino 15.10
Parts:
- added C12: 10uF, Capacitor_SMD:C_0805_2012Metric, F.Cu at (112.5, 115.1)
- added C13: 1uF, Capacitor_SMD:C_0603_1608Metric, F.Cu at (94.8, 120.0)
- added C14: 1uF, Capacitor_SMD:C_0603_1608Metric, F.Cu at (92.5, 120.8)
- added C15: 10uF, Capacitor_SMD:C_0805_2012Metric, F.Cu at (134.6, 125.1)
- added C16: 10uF, Capacitor_SMD:C_0805_2012Metric, F.Cu at (134.6, 83.4)
- added C17: 100nF, Capacitor_SMD:C_0603_1608Metric, F.Cu at (122.6, 110.4)
- added D2: LED_RED, LED_SMD:LED_0603_1608Metric, F.Cu at (143.5, 85.3)
- added D3: LED_Yellow, LED_SMD:LED_0603_1608Metric, F.Cu at (148.1, 85.3)
- added D4: LED_Green, LED_SMD:LED_0603_1608Metric, F.Cu at (152.8, 85.3)
- added R10: 100R, Resistor_SMD:R_0603_1608Metric, F.Cu at (95.6, 122.4)
- added R11: 10K, Resistor_SMD:R_0603_1608Metric, F.Cu at (134.4, 131.5)
- added R12: 10K, Resistor_SMD:R_0603_1608Metric, F.Cu at (134.4, 90.0)
- added R13: 10K, Resistor_SMD:R_0603_1608Metric, F.Cu at (134.4, 128.4)
- added R14: 10K, Resistor_SMD:R_0603_1608Metric, F.Cu at (134.4, 86.8)
- added R15: ?K, Resistor_SMD:R_0603_1608Metric, F.Cu at (143.5, 87.0)
- added R16: ?K, Resistor_SMD:R_0603_1608Metric, F.Cu at (148.1, 87.0)
- added R17: ?K, Resistor_SMD:R_0603_1608Metric, F.Cu at (152.8, 87.0)
- added R6: 10K, Resistor_SMD:R_0603_1608Metric, F.Cu at (118.9, 111.8)
- added R7: 10K, Resistor_SMD:R_0603_1608Metric, F.Cu at (139.1, 91.2)
- added R8: 10K, Resistor_SMD:R_0603_1608Metric, F.Cu at (115.9, 114.9)
- added R9: 10K, Resistor_SMD:R_0603_1608Metric, F.Cu at (97.2, 120.8)
- added SW1: RESET, Button_Switch_THT:SW_PUSH_6mm, F.Cu at (112.0, 112.6)
- added SW2: SW1, Button_Switch_THT:SW_PUSH-12mm, F.Cu at (119.1, 124.0)
- added SW3: SW2, Button_Switch_THT:SW_PUSH-12mm, F.Cu at (119.1, 82.5)
- added U3: 74HC14, Package_SO:SOIC-14_3.9x8.7mm_P1.27mm, F.Cu at (128.1, 112.2)
- moved R1 233.2 mm to (83.0, 87.7)
- moved R2 228.3 mm to (83.1, 85.2)
- moved OLED1 221.6 mm to (88.9, 90.3), turned to 90 degrees
- moved H2 182.9 mm to (153.1, 72.5)
- moved H3 181.3 mm to (153.1, 130.5)
- moved J2 170.0 mm to (146.4, 105.6), turned to 0 degrees
- moved C1 167.1 mm to (146.7, 98.4)
- moved C11 167.1 mm to (132.7, 97.6)
- moved C5 167.1 mm to (129.9, 102.7)
- moved Y1 167.1 mm to (132.4, 102.9)
- moved C10 167.1 mm to (146.7, 100.0)
- moved C6 167.1 mm to (132.5, 105.9)
- moved C7 167.1 mm to (132.8, 99.4)
- moved C8 167.1 mm to (131.3, 95.8)
- moved U1 167.1 mm to (139.6, 98.4)
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Connections:
- U1 pad 10: (no net) -> SW1
- U1 pad 23: (no net) -> LED3
- U1 pad 24: (no net) -> LED2
- U1 pad 25: (no net) -> LED1
- U1 pad 9: (no net) -> SW2
- U2 pad 13: (no net) -> DTR
Routing:
- net +5V: track 0.00 -> 203.1 mm, vias 0 -> 5
- net SDA: track 0.00 -> 61.7 mm, vias 0 -> 2
- net SCL: track 0.00 -> 59.5 mm, vias 0 -> 2
- net RXD: track 0.00 -> 52.6 mm, vias 0 -> 2
- net TXD: track 0.00 -> 51.4 mm
- net ~RESET: track 0.00 -> 46.4 mm, vias 0 -> 2
- net GND: track 0.00 -> 39.7 mm, vias 0 -> 25
- net /IDTR: track 0.00 -> 37.7 mm, vias 0 -> 2
- net /S2: track 0.00 -> 31.4 mm, vias 0 -> 2
- net D+: track 0.00 -> 17.8 mm
- net Net-(R12-Pad1): track 0.00 -> 16.7 mm
- net Net-(R11-Pad1): track 0.00 -> 16.6 mm
- net D-: track 0.00 -> 16.6 mm
- net /S1: track 0.00 -> 16.0 mm
- net SW1: track 0.00 -> 14.9 mm
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Other:
- net class Default: via_dia 0.8 -> 0.6; via_drill 0.4 -> 0.3

Commit message: Finished Protoino
Parts:
- added J3: Conn_02x06_Odd_Even, Connector_PinHeader_2.54mm:PinHeader_2x06_P2.54mm_Vertical, F.Cu at (135.9, 120.5)
- added J4: Conn_02x06_Odd_Even, Connector_PinHeader_2.54mm:PinHeader_2x06_P2.54mm_Vertical, F.Cu at (135.9, 76.8)
- moved H4 10.0 mm to (85.1, 71.5)
- moved H1 10.0 mm to (85.1, 130.5)
- moved C13 8.79 mm to (103.6, 120.5)
- moved C14 8.79 mm to (101.3, 121.2)
- moved C3 8.79 mm to (93.2, 106.7)
- moved C9 8.79 mm to (109.1, 116.9)
- moved D1 8.79 mm to (88.3, 103.9)
- moved F1 8.79 mm to (88.3, 107.6)
- moved FB1 8.79 mm to (88.5, 105.8)
- moved J1 8.79 mm to (84.6, 114.9)
- moved R10 8.79 mm to (104.4, 122.8)
- moved R3 8.79 mm to (93.2, 113.1)
- moved R4 8.79 mm to (93.0, 116.7)
- moved R5 8.79 mm to (91.4, 103.8)
- moved R9 8.79 mm to (105.9, 121.2)
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Connections:
- U1 pad 1: (no net) -> PD3
- U1 pad 11: (no net) -> PD7
- U1 pad 12: (no net) -> PB0
- U1 pad 13: (no net) -> PB1
- U1 pad 14: (no net) -> PB2
- U1 pad 2: (no net) -> PD4
- U1 pad 26: (no net) -> PC3
- U1 pad 32: (no net) -> PD2
Routing:
- net +5V: track 203.1 -> 233.9 mm
- net PD3: track 0.00 -> 24.1 mm, vias 0 -> 1
- net PD4: track 0.00 -> 23.5 mm, vias 0 -> 1
- net PD2: track 0.00 -> 21.8 mm, vias 0 -> 1
- net SCL: track 59.5 -> 80.0 mm, vias 2 -> 3
- net PC3: track 0.00 -> 20.1 mm, vias 0 -> 1
- net PB2: track 0.00 -> 18.6 mm, vias 0 -> 1
- net PB1: track 0.00 -> 17.8 mm, vias 0 -> 1
- net SDA: track 61.7 -> 78.8 mm
- net PB0: track 0.00 -> 17.1 mm, vias 0 -> 1
- net PD7: track 0.00 -> 16.4 mm, vias 0 -> 1
- net RXD: track 52.6 -> 66.6 mm, vias 2 -> 3
- net TXD: track 51.4 -> 62.3 mm, vias 0 -> 1
- net /IDTR: track 37.7 -> 29.1 mm
- net ~RESET: track 46.4 -> 52.4 mm, vias 2 -> 3
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- added copper zone on B.Cu, net GND
- added copper zone on F.Cu, net GND
Other:
- board outline added: 75 x 66 mm
- net class PWR added: clearance 0.2, trace_width 0.4, via_dia 0.6, via_drill 0.3
- board text added: "+5V"
- board text added: "A"
- board text added: "B"
- board text added: "GND"
- board text added: "IU10"
- board text added: "LED1+"
- board text added: "LED2+"
- board text added: "LED3+"
- board text added: "MISO"
- board text added: "MOSI"
- board text added: "PB0"
- board text added: "PB1"
- board text added: "PB2"
- board text added: "PC3"
- board text added: "PD2"
- board text added: "PD3"
- board text added: "PD4"
- board text added: "PD7"
- board text added: "PROTOINO v1.0"
- board text added: "PWR+"
- board text added: "RESET"
- board text added: "RXD"
- board text added: "SCK"
- board text added: "SCL"
- board text added: "SDA"
- board text added: "TXD"
- board text added: "~RESET"
