File: 3_21_22/Protoino01/Protoino01.sch (KiCad schematic (older format))
At the start: 23 parts

Commit message: Protoino - 14.10.2021
Parts:
- added C4: 100nF, Capacitor_SMD:C_0603_1608Metric, symbol Device:C_Small
- added C? (x3): 10uF, Capacitor_SMD:C_0805_2012Metric, symbol Device:C_Small
- added C? (x2): 1uF, Capacitor_SMD:C_0603_1608Metric, symbol Device:C_Small
- added D?: LED_RED, symbol Device:LED_Small_ALT
- added D?: LED_Yellow, symbol Device:LED_Small_ALT
- added D?: LED_Green, symbol Device:LED_Small_ALT
- added H1, H2, H3, H4: MountingHole_Pad, MountingHole:MountingHole_3mm_Pad, symbol Mechanical:MountingHole_Pad
- added J2: ICSP, Connector_PinHeader_2.54mm:PinHeader_2x03_P2.54mm_Vertical, symbol Connector_Generic:Conn_02x03_Odd_Even
- added R? (x3): ?K, Resistor_SMD:R_0603_1608Metric, symbol Device:R_Small
- added R? (x8): 10K, Resistor_SMD:R_0603_1608Metric, symbol Device:R_Small
- added R?: 100R, Resistor_SMD:R_0603_1608Metric, symbol Device:R_Small
- added SW?: RESET, symbol Switch:SW_Push
- added SW?: SW1, symbol Switch:SW_Push
- added SW?: SW2, symbol Switch:SW_Push
- added U? (x6): 74HC14, symbol 74xx:74HC14
- C1, C10, C11, C2, C5, C6, C7, C9: renamed from C?; footprint (none) -> Capacitor_SMD:C_0603_1608Metric
- C3, C8: renamed from C?; footprint (none) -> Capacitor_SMD:C_0805_2012Metric
- D1: renamed from D?; footprint (none) -> LED_SMD:LED_0603_1608Metric
- F1: renamed from F?; footprint (none) -> Fuse:Fuse_0603_1608Metric
- FB1: renamed from FB?; footprint (none) -> Inductor_SMD:L_0805_2012Metric
- J1: renamed from J?; footprint (none) -> Connector_USB:USB_C_Receptacle_HRO_TYPE-C-31-M-12
- R1, R2, R3, R4, R5: renamed from R?; footprint (none) -> Resistor_SMD:R_0603_1608Metric
- Y1: renamed from Y?; footprint (none) -> Crystal:Crystal_SMD_3225-4Pin_3.2x2.5mm
- gave numbers to parts that had none: 3
Connections:
- net +5V: now also D?.2 (A), D?.2 (A), D?.2 (A), J2.2 (Pin_2), R?.2, R?.2, R?.2, R?.2
- net DTR: now also C?.2
- net GND: now also C4.2, C?.1, C?.2, C?.2, C?.2, H1.1, H2.1, H3.1, H4.1, J2.6 (Pin_6), SW?.1, SW?.1, SW?.1
- net LED1: now also R?.1
- net LED2: now also R?.1
- net LED3: now also R?.1
- net MISO: now also J2.1 (Pin_1)
- net MOSI: now also J2.4 (Pin_4)
- net SCK: now also J2.3 (Pin_3)
- net SW1: now also U?.6
- net SW2: now also U?.8
- net ~RESET: now also J2.5 (Pin_5), R?.1, U?.12, U?.4
- net at U2.4 (V3): now also C4.1
- new net: D?.1 (K), R?.2 (x3)
- new net: R?.1, R?.1, SW?.2 (x3)
- new net: C?.1, R?.2, U?.1
- new net: U?.2, U?.3
- new net: C?.1, R?.2, U?.5
- new net: C?.1, R?.2, U?.9
- new net: C?.1, C?.2, R?.1, R?.1
- new net: R?.2, U?.11
- new net: U?.10, U?.13
Other:
- moved on the sheet: C1, C5, C6, R1, R2, U1, U2, Y1

Commit message: protoino 15.10
Parts:
- added C17: 100nF, Capacitor_SMD:C_0603_1608Metric, symbol Device:C_Small
- added unit 7 of U3
- D2, D3, D4: renamed from D?; footprint (none) -> LED_SMD:LED_0603_1608Metric
- SW1: renamed from SW?; footprint (none) -> Button_Switch_THT:SW_PUSH_6mm
- SW2, SW3: renamed from SW?; footprint (none) -> Button_Switch_THT:SW_PUSH-12mm
- U3: renamed from U?; footprint (none) -> Package_SO:SOIC-14_3.9x8.7mm_P1.27mm
- gave numbers to parts that had none: 17
Connections:
- net PC0 is gone; now on net LED3: U1.23 (PC0)
- net PC1 is gone; now on net LED2: U1.24 (PC1)
- net PC2 is gone; now on net LED1: U1.25 (PC2)
- net +5V: now also R12.2, C17.1, U3.14 (VCC)
- net GND: now also C17.2, U3.7 (GND)
- net LED1: no longer U1.32 (PD2)
- net LED2: no longer U1.1 (PD3)
- net LED3: no longer U1.2 (PD4)
- net SW1: now also U1.10 (PD6); no longer U1.9 (PD5)
- net SW2: now also U1.9 (PD5); no longer U1.10 (PD6)
- net IRES: now reaches C12.1, R8.2, U3.1
- net S1: now reaches C15.1, R13.2, U3.5
- net S2: now reaches C16.1, R14.2, U3.9
- net IDTR: now reaches R10.2, U3.11
- new net PD2: U1.32 (PD2)
- new net PD3: U1.1 (PD3)
- new net PD4: U1.2 (PD4)
Other:
- moved on the sheet: U3E, U3F

Commit message: Finished Protoino
Parts:
- added J3, J4: Conn_02x06_Odd_Even, Connector_PinHeader_2.54mm:PinHeader_2x06_P2.54mm_Vertical, symbol Connector_Generic:Conn_02x06_Odd_Even
Connections:
- net +5V: now also J3.1 (Pin_1), J3.5 (Pin_5), J3.9 (Pin_9), J4.10 (Pin_10), J4.2 (Pin_2), J4.6 (Pin_6)
- net GND: now also J3.11 (Pin_11), J3.3 (Pin_3), J3.7 (Pin_7), J4.12 (Pin_12), J4.4 (Pin_4), J4.8 (Pin_8)
- net PB0: now also J3.8 (Pin_8)
- net PB1: now also J3.10 (Pin_10)
- net PB2: now also J3.12 (Pin_12)
- net PC3: now also J4.11 (Pin_11)
- net PD2: now also J4.1 (Pin_1)
- net PD3: now also J3.2 (Pin_2)
- net PD4: now also J3.4 (Pin_4)
- net PD7: now also J3.6 (Pin_6)
- net RXD: now also J4.5 (Pin_5)
- net SCL: now also J4.7 (Pin_7)
- net SDA: now also J4.9 (Pin_9)
- net TXD: now also J4.3 (Pin_3)
Other:
- moved on the sheet: C1, C12, C13, C14, C17, C5, C6, R1, R10, R2, R6, R7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
