File: 3_21_22/12to5Buckconverter/12to5Buckconverter.sch (KiCad schematic (older format))
At the start: 19 parts, among them J1 VIN, J2 VOUT, Q1 AO3401A, U1 TPS5430DDA

Commit message: finished buck converter
Parts:
- removed D?: Red LED, symbol Device:LED
- removed D?: Green Led, symbol Device:LED
- removed R? (x2): R_Small, symbol Device:R_Small
Connections:
- net BOOT: now reaches C1.2, U1.1 (BOOT)
- net EN: now reaches R2.2, R4.1, U1.5 (EN)
- net VIN: now reaches C2.1, C3.1, Q1.2 (S), R2.1, U1.7 (VIN)
- net PH: now reaches C1.1, D1.1 (K), L1.1, U1.8 (PH)
Changed lines of the file:
@@
 Wire Wire Line
 	3100 3050 3450 3050
-$Comp
-L Device:LED D?
-U 1 1 61981F56
-P 5350 4550
-F 0 "D?" V 5389 4432 50  0000 R CNN
-F 1 "Red LED" V 5298 4432 50  0000 R CNN
-F 2 "" H 5350 4550 50  0001 C CNN
-F 3 "~" H 5350 4550 50  0001 C CNN
-	1    5350 4550
-	0    -1   -1   0
-$EndComp
-$Comp
-L Device:LED D?
-U 1 1 61982784
-P 6350 4550
-F 0 "D?" V 6389 4432 50  0000 R CNN
-F 1 "Green Led" V 6298 4432 50  0000 R CNN
-F 2 "" H 6350 4550 50  0001 C CNN
-F 3 "~" H 6350 4550 50  0001 C CNN
-	1    6350 4550
-	0    -1   -1   0
-$EndComp
-$Comp
-L Device:R_Small R?
-U 1 1 61982EC8
-P 5350 4950
-F 0 "R?" H 5409 4996 50  0000 L CNN
-F 1 "R_Small" H 5409 4905 50  0000 L CNN
-F 2 "" H 5350 4950 50  0001 C CNN
-F 3 "~" H 5350 4950 50  0001 C CNN
-	1    5350 4950
-	1    0    0    -1
-$EndComp
-$Comp
-L Device:R_Small R?
-U 1 1 61983311
-P 6350 4950
-F 0 "R?" H 6409 4996 50  0000 L CNN
-F 1 "R_Small" H 6409 4905 50  0000 L CNN
-F 2 "" H 6350 4950 50  0001 C CNN
-F 3 "~" H 6350 4950 50  0001 C CNN
-	1    6350 4950
-	1    0    0    -1
-$EndComp
-Wire Wire Line
-	5350 4850 5350 4700
-Wire Wire Line
-	6350 4850 6350 4700
-Wire Wire Line
-	5350 5050 5350 5150
-Wire Wire Line
-	6350 5050 6350 5150
-$Comp
-L power:GND #PWR?
-U 1 1 61985DE8
-P 5350 5150
-F 0 "#PWR?" H 5350 4900 50  0001 C CNN
-F 1 "GND" H 5355 4977 50  0000 C CNN
-F 2 "" H 5350 5150 50  0001 C CNN
-F 3 "" H 5350 5150 50  0001 C CNN
-	1    5350 5150
-	1    0    0    -1
-$EndComp
-$Comp
-L power:GND #PWR?
-U 1 1 6198611E
-P 6350 5150
-F 0 "#PWR?" H 6350 4900 50  0001 C CNN
-F 1 "GND" H 6355 4977 50  0000 C CNN
-F 2 "" H 6350 5150 50  0001 C CNN
-F 3 "" H 6350 5150 50  0001 C CNN
-	1    6350 5150
-	1    0    0    -1
-$EndComp
-$Comp
-L power:+5V #PWR?
-U 1 1 619864E6
-P 6350 4400
-F 0 "#PWR?" H 6350 4250 50  0001 C CNN
-F 1 "+5V" H 6365 4573 50  0000 C CNN
-F 2 "" H 6350 4400 50  0001 C CNN
-F 3 "" H 6350 4400 50  0001 C CNN
-	1    6350 4400
-	1    0    0    -1
-$EndComp
-$Comp
-L power:+12V #PWR?
-U 1 1 619868C3
-P 5350 4400
-F 0 "#PWR?" H 5350 4250 50  0001 C CNN
-F 1 "+12V" H 5365 4573 50  0000 C CNN
-F 2 "" H 5350 4400 50  0001 C CNN
-F 3 "" H 5350 4400 50  0001 C CNN
-	1    5350 4400
-	1    0    0    -1
-$EndComp
+Text Label 4850 3450 0    50   ~ 0
+EN
+Text Label 4650 3050 0    50   ~ 0
+VIN
+Text Label 6000 3250 0    50   ~ 0
+PH
+Text Label 5950 3050 0    50   ~ 0
+BOOT
 $EndSCHEMATC
