File: 3_21_22/5to12Boostconverter/5to12Boostconverter.sch (KiCad schematic (older format))
At the start: 17 parts, among them J1 5V Connector, J2 12V Connector, U1 TPS61085T

Commit message: Added Homework01_corrected
Connections:
- net +12V: no longer C1.1, C2.1, C3.1, C4.1, C5.1, D1.1 (K), R1.1
- net +5V: no longer C6.1, C7.1, L1.1, U1.3 (EN), U1.6 (IN), U1.7 (FREQ)
- net GND: no longer C1.2, C2.2, C3.2, C4.2, C5.2, C6.2, C7.2, C8.2, C9.2, R3.2, U1.4 (GND)
- net at U1.1 (COMP): no longer R2.1
- net at U1.8 (SS): no longer C8.1
- net at R2.2: no longer C9.1
- now unconnected: D1.2 (A), L1.2, R1.2, R3.1, U1.2 (FB), U1.5 (SW)
Other:
- moved on the sheet: C1, C2, C3, C4, C5, C6, C7, C8, C9, D1, J1, J2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
